File: Robko01_20242009/Robko01_20240920/Robko01_20240920.kicad_sch (KiCad schematic)
At the start: 69 parts, among them J1 Conn_01x04_Pin, J10 Motors, J11 Motors, J12 Conn_01x04_Pin, J13 Conn_01x02_Pin, J14 Conn_01x04_Pin, J15 Conn_01x02_Pin, J16 Conn_01x04_Pin, J17 Conn_01x02_Male, J2 Conn_01x02_Pin, J20 Conn_01x02_Male, J21 Conn_01x19_Pin, J22 Conn_01x19_Pin, J23 Conn_01x06_Pin, J24 Conn_01x04_Pin, J25 Conn_01x04_Pin, J26 Conn_01x04_Pin, J27 Conn_01x06_Pin, J28 Conn_01x02_Male, J29 Conn_01x07_Pin, J3 Conn_01x02_Pin, J30 Conn_01x02_Male, J4 Conn_01x04_Pin, J5 Conn_01x02_Pin, J6 Conn_01x04_Pin, J7 Conn_01x02_Male, J8 Conn_01x02_Pin, J9 Motors, K2 G5V-2, SW1 SW_DIP_x04, SW2 SW_DIP_x04, SW3 SW_DIP_x04, SW4 SW_DIP_x04, SW5 SW_DIP_x04, SW7 SW_DIP_x04, U1 LM7805_TO220

Commit message: Add E-Stop
Parts:
- added J18: Conn_01x02_Male, Connector_PinHeader_2.54mm:PinHeader_1x02_P2.54mm_Horizontal, symbol Robko01-rescue:Conn_01x02_Male-Connector
- added R2: 51k, Resistor_THT:R_Axial_DIN0207_L6.3mm_D2.5mm_P10.16mm_Horizontal, symbol Device:R
- added R3: 15k, Resistor_THT:R_Axial_DIN0207_L6.3mm_D2.5mm_P10.16mm_Horizontal, symbol Device:R
- J1, J12, J14, J16, J4, J6: footprint Connector_PinHeader_2.54mm:PinHeader_1x04_P2.54mm_Vertical -> Connector_PinHeader_2.54mm:PinHeader_1x04_P2.54mm_Horizontal
Connections:
- net GND: now also J18.2 (Pin_2), R3.2
- net VCC: now also R2.1; no longer J17.2 (Pin_2)
- net at A6.3 (1B), J11.8 (Pin_8): now also J16.4 (Pin_4); no longer J16.1 (Pin_1)
- net at A6.4 (1A), J11.7 (Pin_7): now also J16.3 (Pin_3); no longer J16.2 (Pin_2)
- net at A6.5 (2A), J11.6 (Pin_6): now also J16.2 (Pin_2); no longer J16.3 (Pin_3)
- net at A6.6 (2B), J11.5 (Pin_5): now also J16.1 (Pin_1); no longer J16.4 (Pin_4)
- net at A5.3 (1B), J11.12 (Pin_12): now also J14.4 (Pin_4); no longer J14.1 (Pin_1)
- net at A5.4 (1A), J11.11 (Pin_11): now also J14.3 (Pin_3); no longer J14.2 (Pin_2)
- net at A5.5 (2A), J11.10 (Pin_10): now also J14.2 (Pin_2); no longer J14.3 (Pin_3)
- net at A5.6 (2B), J11.9 (Pin_9): now also J14.1 (Pin_1); no longer J14.4 (Pin_4)
- net at A1.3 (1B), J11.4 (Pin_4): now also J1.4 (Pin_4); no longer J1.1 (Pin_1)
- net at A1.4 (1A), J11.3 (Pin_3): now also J1.3 (Pin_3); no longer J1.2 (Pin_2)
- net at A1.5 (2A), J11.2 (Pin_2): now also J1.2 (Pin_2); no longer J1.3 (Pin_3)
- net at A1.6 (2B), J11.1 (Pin_1): now also J1.1 (Pin_1); no longer J1.4 (Pin_4)
- net at A2.3 (1B), J9.1 (Pin_1): now also J4.4 (Pin_4); no longer J4.1 (Pin_1)
- net at A2.4 (1A), J9.2 (Pin_2): now also J4.3 (Pin_3); no longer J4.2 (Pin_2)
- net at A2.5 (2A), J9.3 (Pin_3): now also J4.2 (Pin_2); no longer J4.3 (Pin_3)
- net at A2.6 (2B), J9.4 (Pin_4): now also J4.1 (Pin_1); no longer J4.4 (Pin_4)
- net at A4.3 (1B), J9.12 (Pin_12): now also J12.4 (Pin_4); no longer J12.1 (Pin_1)
- net at A4.4 (1A), J9.11 (Pin_11): now also J12.3 (Pin_3); no longer J12.2 (Pin_2)
- net at A4.5 (2A), J9.10 (Pin_10): now also J12.2 (Pin_2); no longer J12.3 (Pin_3)
- net at A4.6 (2B), J9.9 (Pin_9): now also J12.1 (Pin_1); no longer J12.4 (Pin_4)
- net at A3.3 (1B), J9.5 (Pin_5): now also J6.4 (Pin_4); no longer J6.1 (Pin_1)
- net at A3.4 (1A), J9.6 (Pin_6): now also J6.3 (Pin_3); no longer J6.2 (Pin_2)
- net at A3.5 (2A), J9.7 (Pin_7): now also J6.2 (Pin_2); no longer J6.3 (Pin_3)
- net at A3.6 (2B), J9.8 (Pin_8): now also J6.1 (Pin_1); no longer J6.4 (Pin_4)
- new net: J18.1 (Pin_1), R2.2, R3.1
Other:
- moved on the sheet: J17
