File: hardware/kicad/robko01_retrofit_mb.kicad_pcb (KiCad board)
At the start: 2 copper layers, 178.8 x 143.8 mm, 80 parts, among them J1 Conn_01x04_Pin, J10 Motors, J11 Motors, J12 Conn_01x04_Pin, J13 Conn_01x02_Pin, J14 Conn_01x04_Pin, J15 Conn_01x02_Pin, J16 Conn_01x04_Pin, J17 Conn_01x02_Male, J18 Conn_01x06_Pin, J19 TP-GND, J2 Conn_01x02_Pin, J21 Conn_01x19_Pin, J22 Conn_01x19_Pin, J23 Conn_02x05_Odd_Even, J24 USB_A, J25 USB_B, J28 Conn_01x02_Male, J3 Conn_01x02_Pin, J31 Conn_02x05_Odd_Even, J4 Conn_01x04_Pin, J5 Conn_01x02_Pin, J6 Conn_01x04_Pin, J7 Conn_01x02_Male, J8 Conn_01x02_Pin, J9 Motors, K2 G5V-2, SW1 SW_DIP_x04, SW2 SW_DIP_x04, SW3 SW_DIP_x04, SW4 SW_DIP_x04, SW5 SW_DIP_x04, SW6 RESET, SW7 SW_DIP_x04, U1 LM7805_TO220, U2 PC817

Commit message: Reorganize hardware project and remove dated project naming
Parts:
- JP10: moved to F.Cu
- turned JP10 to 180 degrees
Connections:
- J11 pad 13: GPIO35 -> M6-Limit
- J11 pad 3: unconnected-(J11-Pin_3-Pad3) -> Net-(A1-1A)
Routing:
- net VSPI_MISO: track 238.4 -> 161.0 mm
- net VSPI_MOSI: track 243.5 -> 169.7 mm
- net M6-Limit: track 340.6 -> 342.1 mm
Other:
- board text added: "Base"
- board text added: "Black"
- board text added: "Elbow"
- board text added: "Green"
- board text added: "Gripper"
- board text added: "Red"
- board text added: "Shoulder"
- board text added: "White"
