File: hardware/kicad/robko01_retrofit_mb.kicad_pcb (KiCad board)
At the start: 2 copper layers, 178.8 x 143.8 mm, 84 parts, among them J1 Conn_01x04_Pin, J10 Motors, J11 Motors, J12 Conn_01x04_Pin, J13 Conn_01x02_Pin, J14 Conn_01x04_Pin, J15 Conn_01x02_Pin, J16 Conn_01x04_Pin, J17 Conn_01x02_Male, J18 Conn_01x06_Pin, J19 TP-GND, J2 Conn_01x02_Pin, J21 Conn_01x19_Pin, J22 Conn_01x19_Pin, J23 Conn_02x05_Odd_Even, J24 USB_A, J25 USB_B, J28 Conn_01x02_Male, J3 Conn_01x02_Pin, J31 Conn_02x05_Odd_Even, J4 Conn_01x04_Pin, J5 Conn_01x02_Pin, J6 Conn_01x04_Pin, J7 Conn_01x02_Male, J8 Conn_01x02_Pin, J9 Motors, K2 G5V-2, SW1 SW_DIP_x04, SW2 SW_DIP_x04, SW3 SW_DIP_x04, SW4 SW_DIP_x04, SW5 SW_DIP_x04, SW6 RESET, SW7 SW_DIP_x04, U1 LM7805_TO220, U2 PC817

Commit message: Convert electrolytic capacitors to SMD with local 3D model
Parts:
- C10, C12, C14, C4, C6, C8: footprint Capacitor_THT:CP_Radial_D8.0mm_P3.50mm -> Capacitor_SMD:CP_Elec_8x10.5
- moved C10 3.73 mm to (172.8, 112.6)
- moved C12 3.73 mm to (172.8, 90.1)
- moved C14 3.73 mm to (172.8, 67.6)
- moved C8 3.73 mm to (172.8, 135.1)
- moved C4 3.73 mm to (172.8, 45.1)
- moved C6 3.73 mm to (172.8, 22.6)
Routing:
- net Net-(A6-VMOT): track 28.9 -> 35.8 mm, vias 1 -> 2
- net Net-(A5-VMOT): track 28.7 -> 35.6 mm, vias 1 -> 2
- net Net-(A4-VMOT): track 29.0 -> 35.8 mm, vias 1 -> 2
- net Net-(A1-VMOT): track 31.7 -> 38.5 mm, vias 1 -> 2
- net Net-(A2-VMOT): track 28.4 -> 35.3 mm, vias 1 -> 2
- net Net-(A3-VMOT): track 29.0 -> 35.9 mm, vias 1 -> 2
