File: hardware/kicad/robko01_retrofit_mb.kicad_sch (KiCad schematic)
At the start: 80 parts, among them J1 Conn_01x04_Pin, J10 Motors, J11 Motors, J12 Conn_01x04_Pin, J13 Conn_01x02_Pin, J14 Conn_01x04_Pin, J15 Conn_01x02_Pin, J16 Conn_01x04_Pin, J17 Conn_01x02_Male, J18 Conn_01x06_Pin, J19 TP-GND, J2 Conn_01x02_Pin, J21 Conn_01x19_Pin, J22 Conn_01x19_Pin, J23 Conn_02x05_Odd_Even, J24 USB_A, J25 USB_B, J28 Conn_01x02_Male, J3 Conn_01x02_Pin, J31 Conn_02x05_Odd_Even, J4 Conn_01x04_Pin, J5 Conn_01x02_Pin, J6 Conn_01x04_Pin, J7 Conn_01x02_Male, J8 Conn_01x02_Pin, J9 Motors, K2 G5V-2, SW1 SW_DIP_x04, SW2 SW_DIP_x04, SW3 SW_DIP_x04, SW4 SW_DIP_x04, SW5 SW_DIP_x04, SW6 RESET, SW7 SW_DIP_x04, U1 LM7805_TO220, U2 PC817

Commit message: Reorganize hardware project and remove dated project naming
Connections:
- net GPIO35 is gone; now on net M6-Limit: J11.13 (Pin_13)
- net at A1.4 (1A), J1.3 (Pin_3): now also J11.3 (Pin_3)

Commit message: Convert ceramic capacitors to 0805 footprints
Parts:
- C1, C11, C13, C2, C3, C5, C7, C9: footprint Capacitor_THT:C_Disc_D7.0mm_W2.5mm_P5.00mm -> Capacitor_SMD:C_0805_2012Metric
Changed lines of the file:
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@@
 			)
 		)
-		(property "Footprint" "Capacitor_THT:C_Disc_D7.0mm_W2.5mm_P5.00mm"
+		(property "Footprint" "Capacitor_SMD:C_0805_2012Metric"
 			(at 721.0552 614.68 0)
 			(effects
@@
 			)
 		)
-		(property "Footprint" "Capacitor_THT:C_Disc_D7.0mm_W2.5mm_P5.00mm"
+		(property "Footprint" "Capacitor_SMD:C_0805_2012Metric"
 			(at 719.7852 307.34 0)
 			(effects
@@
 			)
 		)
-		(property "Footprint" "Capacitor_THT:C_Disc_D7.0mm_W2.5mm_P5.00mm"
+		(property "Footprint" "Capacitor_SMD:C_0805_2012Metric"
 			(at 721.0552 539.75 0)
 			(effects
@@
 			)
 		)
-		(property "Footprint" "Capacitor_THT:C_Disc_D7.0mm_W2.5mm_P5.00mm"
+		(property "Footprint" "Capacitor_SMD:C_0805_2012Metric"
 			(at 719.7852 232.41 0)
 			(effects
@@
 			)
 		)
-		(property "Footprint" "Capacitor_THT:C_Disc_D7.0mm_W2.5mm_P5.00mm"
+		(property "Footprint" "Capacitor_SMD:C_0805_2012Metric"
 			(at 719.7852 389.89 0)
 			(effects
@@
 			)
 		)
-		(property "Footprint" "Capacitor_THT:C_Disc_D7.0mm_W2.5mm_P5.00mm"
+		(property "Footprint" "Capacitor_SMD:C_0805_2012Metric"
 			(at 383.2352 350.52 0)
 			(effects
@@
 			)
 		)
-		(property "Footprint" "Capacitor_THT:C_Disc_D7.0mm_W2.5mm_P5.00mm"
+		(property "Footprint" "Capacitor_SMD:C_0805_2012Metric"
 			(at 407.3652 350.52 0)
 			(effects
@@
 			)
 		)
-		(property "Footprint" "Capacitor_THT:C_Disc_D7.0mm_W2.5mm_P5.00mm"
+		(property "Footprint" "Capacitor_SMD:C_0805_2012Metric"
 			(at 719.7852 464.82 0)
 			(effects

Commit message: Convert D1 and D2 to SMD and remove obsolete BOM snapshots
Parts:
- D1, D2: value 1N4007 -> S1M; footprint Diode_THT:D_DO-41_SOD81_P10.16mm_Horizontal -> Diode_SMD:D_SMA; symbol Diode:1N4007 -> Device:D
Changed lines of the file:
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@@
 	)
 	(symbol
-		(lib_id "Diode:1N4007")
+		(lib_id "Device:D")
 		(at 322.58 345.44 270)
 		(unit 1)
@@
 			)
 		)
-		(property "Value" "1N4007"
+		(property "Value" "S1M"
 			(at 325.12 346.7099 90)
 			(effects
@@
 			)
 		)
-		(property "Footprint" "Diode_THT:D_DO-41_SOD81_P10.16mm_Horizontal"
+		(property "Footprint" "Diode_SMD:D_SMA"
 			(at 318.135 345.44 0)
 			(effects
@@
 			)
 		)
-		(property "Datasheet" "http://www.vishay.com/docs/88503/1n4001.pdf"
+		(property "Datasheet" "https://www.vishay.com/doc/?88711="
 			(at 322.58 345.44 0)
 			(effects
@@
 			)
 		)
-		(property "Description" "1000V 1A General Purpose Rectifier Diode, DO-41"
+		(property "Description" "1000V 1A surface-mount rectifier diode, SMA (DO-214AC)"
 			(at 322.58 345.44 0)
 			(effects
@@
 	)
 	(symbol
-		(lib_id "Diode:1N4007")
+		(lib_id "Device:D")
 		(at 322.58 328.93 90)
 		(unit 1)
@@
 			)
 		)
-		(property "Value" "1N4007"
+		(property "Value" "S1M"
 			(at 325.12 330.1999 90)
 			(effects
@@
 			)
 		)
-		(property "Footprint" "Diode_THT:D_DO-41_SOD81_P10.16mm_Horizontal"
+		(property "Footprint" "Diode_SMD:D_SMA"
 			(at 327.025 328.93 0)
 			(effects
@@
 			)
 		)
-		(property "Datasheet" "http://www.vishay.com/docs/88503/1n4001.pdf"
+		(property "Datasheet" "https://www.vishay.com/doc/?88711="
 			(at 322.58 328.93 0)
 			(effects
@@
 			)
 		)
-		(property "Description" "1000V 1A General Purpose Rectifier Diode, DO-41"
+		(property "Description" "1000V 1A surface-mount rectifier diode, SMA (DO-214AC)"
 			(at 322.58 328.93 0)
 			(effects

Commit message: Convert resistors to 0805 and split RN1 into five 10k resistors
Parts:
- removed RN1: R_Network05, Resistor_THT:R_Array_SIP6, symbol Device:R_Network05
- added R3, R4, R5, R6, R7: 10k, Resistor_SMD:R_0805_2012Metric, symbol Device:R_Small
- R1, R2: footprint Resistor_THT:R_Axial_DIN0207_L6.3mm_D2.5mm_P10.16mm_Horizontal -> Resistor_SMD:R_0805_2012Metric
Connections:
- net +3.3V: now also R3.1, R4.1, R5.1, R6.1, R7.1
- net E-STOP: now also R7.2
- net M1-Limit: now also R5.2
- net M2-Limit: now also R4.2
- net M3-Limit: now also R3.2
- net M6-Limit: now also R6.2

Commit message: Convert D3 and D4 to 0805 LED footprints
Parts:
- D3: value LED 3mm Green -> LED 0805 Green; footprint LED_THT:LED_D5.0mm -> LED_SMD:LED_0805_2012Metric
- D4: value LED 3mm Red -> LED 0805 Red; footprint LED_THT:LED_D5.0mm -> LED_SMD:LED_0805_2012Metric
Changed lines of the file:
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@@
 			)
 		)
-		(property "Value" "LED 3mm Green"
+		(property "Value" "LED 0805 Green"
 			(at 289.56 348.2974 90)
 			(effects
@@
 			)
 		)
-		(property "Footprint" "LED_THT:LED_D5.0mm"
+		(property "Footprint" "LED_SMD:LED_0805_2012Metric"
 			(at 285.75 345.44 0)
 			(effects
@@
 			)
 		)
-		(property "Value" "LED 3mm Red"
+		(property "Value" "LED 0805 Red"
 			(at 300.99 345.1224 90)
 			(effects
@@
 			)
 		)
-		(property "Footprint" "LED_THT:LED_D5.0mm"
+		(property "Footprint" "LED_SMD:LED_0805_2012Metric"
 			(at 298.45 345.44 0)
 			(effects

Commit message: Convert electrolytic capacitors to SMD with local 3D model
Parts:
- C10, C12, C14, C4, C6, C8: footprint Capacitor_THT:CP_Radial_D8.0mm_P3.50mm -> Capacitor_SMD:CP_Elec_8x10.5
Changed lines of the file:
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@@
 			)
 		)
-		(property "Footprint" "Capacitor_THT:CP_Radial_D8.0mm_P3.50mm"
+		(property "Footprint" "Capacitor_SMD:CP_Elec_8x10.5"
 			(at 731.2152 307.34 0)
 			(effects
@@
 			)
 		)
-		(property "Footprint" "Capacitor_THT:CP_Radial_D8.0mm_P3.50mm"
+		(property "Footprint" "Capacitor_SMD:CP_Elec_8x10.5"
 			(at 732.4852 614.68 0)
 			(effects
@@
 			)
 		)
-		(property "Footprint" "Capacitor_THT:CP_Radial_D8.0mm_P3.50mm"
+		(property "Footprint" "Capacitor_SMD:CP_Elec_8x10.5"
 			(at 731.2152 389.89 0)
 			(effects
@@
 			)
 		)
-		(property "Footprint" "Capacitor_THT:CP_Radial_D8.0mm_P3.50mm"
+		(property "Footprint" "Capacitor_SMD:CP_Elec_8x10.5"
 			(at 731.2152 464.82 0)
 			(effects
@@
 			)
 		)
-		(property "Footprint" "Capacitor_THT:CP_Radial_D8.0mm_P3.50mm"
+		(property "Footprint" "Capacitor_SMD:CP_Elec_8x10.5"
 			(at 732.4852 539.75 0)
 			(effects
@@
 			)
 		)
-		(property "Footprint" "Capacitor_THT:CP_Radial_D8.0mm_P3.50mm"
+		(property "Footprint" "Capacitor_SMD:CP_Elec_8x10.5"
 			(at 731.2152 232.41 0)
 			(effects
